File: Boost_Converter/Boost_Converter/Boost_Converter/Boost_Converter.kicad_pcb (KiCad board)
At the start: 2 copper layers, 100 x 88 mm, 27 parts, among them J1 USB_A, J2 USB_B_Micro, U1 MC34063A-E, U2 DIO5158, U3 NC7SZ86M5X

Commit message: Add files via upload
FInal update files
Routing:
- net GND: vias 2 -> 80
- added copper zone on B.Cu, net GND
Other:
- board text added: "Two Liion Cell Buck Boost Converter 5V 1A |Power bank|"
- board text added: "https://github.com/skndungu/Two-Cell-Liion-Buck-Boost-Conveter-output-5V-1A"
- board text added: "© 2019"
- board text removed: "Two Liion Cell Buck Boost Converter 5V 1.5A |Power bank|"
- board text removed: "https://github.com/skndungu/Two-Cell-Liion-Buck-Boost-Conveter-output-5V-1.5A"
Changed lines of the file:
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@@
   (general
     (thickness 1.6)
-    (drawings 11)
-    (tracks 157)
+    (drawings 12)
+    (tracks 235)
     (zones 0)
     (modules 27)
@@
     (via_min_size 0.4)
     (via_min_drill 0.3)
+    (user_via 1.6 0.5)
     (uvia_size 0.3)
     (uvia_drill 0.1)
@@
     (visible_elements FFFFEF7F)
     (pcbplotparams
-      (layerselection 0x010fc_ffffffff)
+      (layerselection 0x3d0fc_ffffffff)
       (usegerberextensions false)
       (usegerberattributes false)
@@
       (outputformat 1)
       (mirror false)
-      (drillshape 1)
+      (drillshape 0)
       (scaleselection 1)
-      (outputdirectory ""))
+      (outputdirectory "../../gerber/"))
   )
   (net 0 "")
@@
     )
   )
+  (gr_text " © 2019" (at 101.75 33.25) (layer F.SilkS)
+    (effects (font (size 1 1) (thickness 0.15)))
+  )
   (gr_text https://www.skndungudevs.com/ (at 111 38.25) (layer F.SilkS)
     (effects (font (size 1 1) (thickness 0.15)))
   )
-  (gr_text https://github.com/skndungu/Two-Cell-Liion-Buck-Boost-Conveter-output-5V-1.5A (at 110.75 109.75) (layer F.SilkS)
+  (gr_text https://github.com/skndungu/Two-Cell-Liion-Buck-Boost-Conveter-output-5V-1A (at 110.75 109.75) (layer F.SilkS)
     (effects (font (size 0.5 0.5) (thickness 0.1)))
   )
@@
     (effects (font (size 1 1) (thickness 0.15)))
   )
-  (gr_text "Two Liion Cell Buck Boost Converter 5V 1.5A\n|Power bank|" (at 110.25 35.5) (layer F.SilkS)
+  (gr_text "Two Liion Cell Buck Boost Converter 5V 1A\n|Power bank|" (at 110.25 35.5) (layer F.SilkS)
     (effects (font (size 0.8 0.8) (thickness 0.15)))
   )
@@
   (segment (start 30.325 76.8) (end 30.025 76.5) (width 0.25) (layer F.Cu) (net 2))
   (segment (start 32.725 76.8) (end 30.325 76.8) (width 0.25) (layer F.Cu) (net 2))
+  (via (at 93.25 32.5) (size 1.5) (drill 0.4) (layers F.Cu B.Cu) (net 2))
+  (via (at 97.5 62.5) (size 0.8) (drill 0.4) (layers F.Cu B.Cu) (net 2))
+  (via (at 97.5 63.75) (size 0.8) (drill 0.4) (layers F.Cu B.Cu) (net 2))
+  (via (at 94.25 67.75) (size 0.8) (drill 0.4) (layers F.Cu B.Cu) (net 2))
+  (via (at 95.75 66.25) (size 0.8) (drill 0.4) (layers F.Cu B.Cu) (net 2))
+  (via (at 96 62.5) (size 0.8) (drill 0.4) (layers F.Cu B.Cu) (net 2))
+  (via (at 99 94) (size 0.8) (drill 0.4) (layers F.Cu B.Cu) (net 2))
+  (via (at 99 90.25) (size 0.8) (drill 0.4) (layers F.Cu B.Cu) (net 2))
+  (via (at 89.25 94.5) (size 0.8) (drill 0.4) (layers F.Cu B.Cu) (net 2))
+  (via (at 36.75 80.75) (size 0.8) (drill 0.4) (layers F.Cu B.Cu) (net 2))
+  (via (at 35 78.75) (size 0.8) (drill 0.4) (layers F.Cu B.Cu) (net 2))
+  (via (at 91 49) (size 0.8) (drill 0.4) (layers F.Cu B.Cu) (net 2))
+  (via (at 91.25 56.25) (size 1.6) (drill 0.5) (layers F.Cu B.Cu) (net 2))
+  (via (at 92.75 53.25) (size 1.6) (drill 0.5) (layers F.Cu B.Cu) (net 2))
+  (via (at 92.75 58) (size 1.6) (drill 0.5) (layers F.Cu B.Cu) (net 2))
+  (via (at 30 81.25) (size 1.6) (drill 0.5) (layers F.Cu B.Cu) (net 2))
+  (via (at 30 84.75) (size 1.6) (drill 0.5) (layers F.Cu B.Cu) (net 2))
+  (via (at 30 88.25) (size 1.6) (drill 0.5) (layers F.Cu B.Cu) (net 2))
+  (via (at 30 91.75) (size 1.6) (drill 0.5) (layers F.Cu B.Cu) (net 2))
+  (via (at 30 95.5) (size 1.6) (drill 0.5) (layers F.Cu B.Cu) (net 2))
+  (via (at 30 98.75) (size 1.6) (drill 0.5) (layers F.Cu B.Cu) (net 2))
+  (via (at 30 102.5) (size 1.6) (drill 0.5) (layers F.Cu B.Cu) (net 2))
+  (via (at 30 107.5) (size 1.6) (drill 0.5) (layers F.Cu B.Cu) (net 2))
+  (via (at 30 112.75) (size 1.6) (drill 0.5) (layers F.Cu B.Cu) (net 2))
+  (via (at 30 117.75) (size 1.6) (drill 0.5) (layers F.Cu B.Cu) (net 2))
+  (via (at 30.25 68) (size 1.6) (drill 0.5) (layers F.Cu B.Cu) (net 2))
+  (via (at 30.25 61.75) (size 1.6) (drill 0.5) (layers F.Cu B.Cu) (net 2))
+  (via (at 30.25 56.5) (size 1.6) (drill 0.5) (layers F.Cu B.Cu) (net 2))
+  (via (at 30.25 50.75) (size 1.6) (drill 0.5) (layers F.Cu B.Cu) (net 2))
+  (via (at 30.25 45.25) (size 1.6) (drill 0.5) (layers F.Cu B.Cu) (net 2))
+  (via (at 30.25 39.25) (size 1.6) (drill 0.5) (layers F.Cu B.Cu) (net 2))
+  (via (at 30.25 33.5) (size 1.6) (drill 0.5) (layers F.Cu B.Cu) (net 2))
+  (via (at 52.75 41.25) (size 1.6) (drill 0.5) (layers F.Cu B.Cu) (net 2))
+  (via (at 57 34.5) (size 1.6) (drill 0.5) (layers F.Cu B.Cu) (net 2))
+  (via (at 47.25 34.25) (size 1.6) (drill 0.5) (layers F.Cu B.Cu) (net 2))
+  (via (at 71.75 34) (size 1.6) (drill 0.5) (layers F.Cu B.Cu) (net 2))
+  (via (at 82.5 34) (size 1.6) (drill 0.5) (layers F.Cu B.Cu) (net 2))
+  (via (at 77.25 40.75) (size 1.6) (drill 0.5) (layers F.Cu B.Cu) (net 2))
+  (via (at 96.75 44.5) (size 1.6) (drill 0.5) (layers F.Cu B.Cu) (net 2))
+  (via (at 103.25 44.5) (size 1.6) (drill 0.5) (layers F.Cu B.Cu) (net 2))
+  (via (at 112.5 44.5) (size 1.6) (drill 0.5) (layers F.Cu B.Cu) (net 2))
+  (via (at 122 44.5) (size 1.6) (drill 0.5) (layers F.Cu B.Cu) (net 2))
+  (via (at 125 50.25) (size 1.6) (drill 0.5) (layers F.Cu B.Cu) (net 2))
+  (via (at 125 57) (size 1.6) (drill 0.5) (layers F.Cu B.Cu) (net 2))
+  (via (at 125 62.25) (size 1.6) (drill 0.5) (layers F.Cu B.Cu) (net 2))
+  (via (at 118.25 61.5) (size 1.6) (drill 0.5) (layers F.Cu B.Cu) (net 2))
+  (via (at 118.75 74.25) (size 1.6) (drill 0.5) (layers F.Cu B.Cu) (net 2))
+  (via (at 118.75 69) (size 1.6) (drill 0.5) (layers F.Cu B.Cu) (net 2))
+  (via (at 118.25 81.75) (size 1.6) (drill 0.5) (layers F.Cu B.Cu) (net 2))
+  (via (at 125.5 81.5) (size 1.6) (drill 0.5) (layers F.Cu B.Cu) (net 2))
+  (via (at 125.5 86.25) (size 1.6) (drill 0.5) (layers F.Cu B.Cu) (net 2))
+  (via (at 125.5 91) (size 1.6) (drill 0.5) (layers F.Cu B.Cu) (net 2))
+  (via (at 125.5 96) (size 1.6) (drill 0.5) (layers F.Cu B.Cu) (net 2))
+  (via (at 117.25 99.5) (size 1.6) (drill 0.5) (layers F.Cu B.Cu) (net 2))
+  (via (at 125.5 99.5) (size 1.6) (drill 0.5) (layers F.Cu B.Cu) (net 2))
+  (via (at 125.5 104.25) (size 1.6) (drill 0.5) (layers F.Cu B.Cu) (net 2))
+  (via (at 125.5 107.75) (size 1.6) (drill 0.5) (layers F.Cu B.Cu) (net 2))
+  (via (at 125.5 112.5) (size 1.6) (drill 0.5) (layers F.Cu B.Cu) (net 2))
+  (via (at 125.5 117) (size 1.6) (drill 0.5) (layers F.Cu B.Cu) (net 2))
+  (via (at 94.5 116) (size 1.6) (drill 0.5) (layers F.Cu B.Cu) (net 2))
+  (via (at 104.5 116) (size 1.6) (drill 0.5) (layers F.Cu B.Cu) (net 2))
+  (via (at 113.75 116) (size 1.6) (drill 0.5) (layers F.Cu B.Cu) (net 2))
+  (via (at 120.75 116.5) (size 1.6) (drill 0.5) (layers F.Cu B.Cu) (net 2))
+  (via (at 37 89) (size 1.6) (drill 0.5) (layers F.Cu B.Cu) (net 2))
+  (via (at 37.25 97.75) (size 1.6) (drill 0.5) (layers F.Cu B.Cu) (net 2))
+  (via (at 36.75 108.75) (size 1.6) (drill 0.5) (layers F.Cu B.Cu) (net 2))
+  (via (at 37.75 47.5) (size 1.6) (drill 0.5) (layers F.Cu B.Cu) (net 2))
+  (via (at 37.5 60) (size 1.6) (drill 0.5) (layers F.Cu B.Cu) (net 2))
+  (via (at 113.75 53.25) (size 1.6) (drill 0.5) (layers F.Cu B.Cu) (net 2))
+  (via (at 118.25 57) (size 1.6) (drill 0.5) (layers F.Cu B.Cu) (net 2))
+  (via (at 91.75 40) (size 1.6) (drill 0.5) (layers F.Cu B.Cu) (net 2))
+  (via (at 100 100.75) (size 1.6) (drill 0.5) (layers F.Cu B.Cu) (net 2))
+  (via (at 116 88.5) (size 1.6) (drill 0.5) (layers F.Cu B.Cu) (net 2))
+  (via (at 110 103.25) (size 1.6) (drill 0.5) (layers F.Cu B.Cu) (net 2))
+  (via (at 100.25 107) (size 1.6) (drill 0.5) (layers F.Cu B.Cu) (net 2))
+  (via (at 107.5 48.25) (size 1.6) (drill 0.5) (layers F.Cu B.Cu) (net 2))
+  (via (at 124.75 39.5) (size 1.6) (drill 0.5) (layers F.Cu B.Cu) (net 2))
+  (via (at 125.25 32.75) (size 1.6) (drill 0.5) (layers F.Cu B.Cu) (net 2))
   (segment (start 97.87929 55.12929) (end 98.75 56) (width 0.55) (layer F.Cu) (net 3))
   (segment (start 97.47499 54.72499) (end 97.87929 55.12929) (width 0.55) (layer F.Cu) (net 3))
@@
       )
     )
+  )
+  (zone (net 2) (net_name GND) (layer B.Cu) (hatch edge 0.508)
+    (connect_pads (clearance 0.508))
+    (min_thickness 0.254)
+    (fill yes (arc_segments 32) (thermal_gap 0.508) (thermal_bridge_width 0.508))
+    (polygon
+      (pts
+        (xy 28 31) (xy 128.25 31) (xy 128 119) (xy 28 119)
+      )
+    )
