File: Boost_Converter/Boost_Converter/Boost_Converter/Boost_Converter.sch (KiCad schematic (older format))
At the start: 26 parts, among them J1 USB_A, J2 USB_B_Micro, U1 MC34063A-E, U2 DIO5158, U3 NC7SZ86M5X

Commit message: Add files via upload
FInal update files
Other:
- note added: "Open Source Hardware"
- note added: "Resources: https://github.com/skndungu/Two-Cell-Liion-Buck-Boost-Conveter-output-5V-1.5A"
Changed lines of the file:
@@
 Comment1 ""
 Comment2 ""
-Comment3 ""
+Comment3 "Licence: CERN OHL"
 Comment4 "Author:  Simon Ndungu"
 $EndDescr
@@
 L Graphic:Logo_Open_Hardware_Small #LOGO2
 U 1 1 5D4B6FE2
-P 8700 6750
-F 0 "#LOGO2" H 8700 7025 50  0001 C CNN
-F 1 "Logo_Open_Hardware_Small" H 8700 6525 50  0001 C CNN
-F 2 "" H 8700 6750 50  0001 C CNN
-F 3 "~" H 8700 6750 50  0001 C CNN
-	1    8700 6750
+P 10950 6750
+F 0 "#LOGO2" H 10950 7025 50  0001 C CNN
+F 1 "Logo_Open_Hardware_Small" H 10950 6525 50  0001 C CNN
+F 2 "" H 10950 6750 50  0001 C CNN
+F 3 "~" H 10950 6750 50  0001 C CNN
+	1    10950 6750
 	1    0    0    -1
 $EndComp
@@
 	1    0    0    -1
 $EndComp
+Text Notes 7000 6900 0    47   ~ 0
+Resources: https://github.com/skndungu/Two-Cell-Liion-Buck-Boost-Conveter-output-5V-1.5A
+Text Notes 3750 5200 0    50   ~ 0
+Open Source Hardware
 $EndSCHEMATC
